File: KiCad/Linky_Tempo_HomeKit.kicad_pcb (KiCad board)
At the start: 2 copper layers, 111.8 x 78.7 mm, 21 parts, among them J1 TIC, J3 Main(1) + Fil pilote (3,5,7), J4 +3.3V, J5 GND, J6 SCL, J7 SDA, Q1 BS170, Q2 PN2222A, SW1 Setup, SW2 Annul_Délestage, U2 LTV-814, U3 MOC3041M

Commit message: corrections diverses
Parts:
- removed Q1: BS170, Package_TO_SOT_THT:TO-92_Inline_Wide
- added Q3: 2N7000, Package_TO_SOT_THT:TO-92_Inline, F.Cu at (165.1, 100.3)
- R2: footprint Resistor_THT:R_Axial_DIN0207_L6.3mm_D2.5mm_P5.08mm_Vertical -> Resistor_THT:R_Axial_DIN0207_L6.3mm_D2.5mm_P2.54mm_Vertical
Routing:
- net Net-(Q3-D): track 21.4 -> 27.2 mm, vias 0 -> 2
- net Net-(Q3-G): track 16.3 -> 15.2 mm
- net GND: track 191.6 -> 192.4 mm
Other:
- board text added: "220V"
