File: KiCad/Linky_Tempo_HomeKit.kicad_sch (KiCad schematic)
At the start: 21 parts, among them J1 TIC, J3 Main(1) + Fil pilote (3,5,7), J4 +3.3V, J5 GND, J6 SCL, J7 SDA, Q1 BS170, Q2 PN2222A, SW1 Setup, SW2 Annul_Délestage, U2 LTV-814, U3 MOC3041M

Commit message: corrections diverses
Parts:
- removed Q1: BS170, Package_TO_SOT_THT:TO-92_Inline_Wide, symbol Transistor_FET:BS170
- added Q3: 2N7000, Package_TO_SOT_THT:TO-92_Inline, symbol Transistor_FET:2N7000
- R2: footprint Resistor_THT:R_Axial_DIN0207_L6.3mm_D2.5mm_P5.08mm_Vertical -> Resistor_THT:R_Axial_DIN0207_L6.3mm_D2.5mm_P2.54mm_Vertical
Connections:
- net GND: now also Q3.1 (S)
- net at R3.2, U1.21 (GPIO16=RX2): now also Q3.3 (D)
- net at R2.2, U2.3: now also Q3.2 (G)
